Commit message: Add transmissions and ros_gazebo_control plugin to URDF

File: urdf/doggo_description.urdf (robot description, URDF)
Before this commit: robot doggo_description, 22 links, 21 joints
Links:
- link base_link: geometry collision mesh filename=package://doggo_description/meshes/base_link.; visual mesh filename=package://doggo_description/meshes/base_link.

Commit message: Add updated urdf with SDF tags for mimicing parallel joints

File: urdf/doggo_description.urdf (robot description, URDF)
Before this commit: robot doggo_description, 22 links, 21 joints
Links:
- added link footstep1
- added link footstep2
- added link footstep3
- added link footstep4
Joints:
- added joint shoe1_footstep1: type fixed, parent shoe1, child footstep1, origin xyz=0 -0.19 0 rpy=0 2.13 1.5708, axis 0 0 0
- added joint shoe2_footstep2: type fixed, parent shoe2, child footstep2, origin xyz=0 -0.19 0 rpy=0 1.011 1.5708, axis 0 0 0
- added joint shoe3_footstep3: type fixed, parent shoe3, child footstep3, origin xyz=0 -0.19 0 rpy=0 1.011 1.5708, axis 0 0 0
- added joint shoe4_footstep4: type fixed, parent shoe4, child footstep4, origin xyz=0 -0.19 0 rpy=0 2.13 1.5708, axis 0 0 0
