Commit message: Add Modidied meshes and URDF

File: urdf/doggo_description_with_rgbd_camera.urdf (robot description, URDF)
Before this commit: robot doggo_description, 26 links, 25 joints
Links:
- added link camera_depth_frame
- added link camera_link, mass 1e-5; collision mesh filename=package://doggo_description/meshes/realsense_d435.STL; visual mesh filename=package://doggo_description/meshes/realsense_d435.STL
Joints:
- added joint cam_joint: type fixed, parent base_link, child camera_depth_frame, origin xyz=0.25 0.0 0.1 rpy=0 1 0
- added joint cam_joint1: type fixed, parent base_link, child camera_link, origin xyz=0.25 0.0 0.1 rpy=0 1 0
